Commit message: r2d2 with camera

File: src/my_r2d2/urdf/r2d2.urdf.xacro (robot description, xacro)
@@ -220,3 +220,10 @@
     <origin xyz="0 0 ${(0.6-0.25)+wheeldiam+(0.1/2)}" />
   </joint>
+  <link name="eye">
+  </link>
+  <joint name="box_to_eye" type="fixed">
+    <parent link="box"/>
+    <child link="eye"/>
+    <origin rpy="-${pi/2} 0 -${pi/2}" xyz="0 0 0"/>
+  </joint>
 </robot>
